File: ClapLamp.kicad_sch (KiCad schematic)
At the start: 26 parts, among them J2 Jack-DC, U1 ESP32-C3-DevKitM-1

Commit message: Add files via upload
Connections:
- net at D20.1 (DOUT): now also D19.1 (DOUT)
- net at D17.1 (DOUT): now also D18.1 (DOUT)
- new net: D4.2 (DIN), D7.2 (DIN)
- new net: D1.2 (DIN), R1.1
- now unconnected: D10.2 (DIN)
Changed lines of the file:
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@@
-	)
-	(junction
-		(at 118.11 86.36)
-		(diameter 0)
-		(color 0 0 0 0)
 	)
 	(junction
@@
 	)
 	(junction
-		(at 118.11 67.31)
-		(diameter 0)
-		(color 0 0 0 0)
-	)
-	(junction
 		(at 196.85 74.93)
 		(diameter 0)
@@
 	)
 	(junction
-		(at 118.11 105.41)
-		(diameter 0)
-		(color 0 0 0 0)
-	)
-	(junction
 		(at 173.99 116.84)
 		(diameter 0)
@@
 	(wire
 		(pts
-			(xy 118.11 105.41) (xy 148.59 105.41)
+			(xy 148.59 86.36) (xy 146.05 86.36)
 		)
 		(stroke
@@
 	(wire
 		(pts
+			(xy 245.11 105.41) (xy 247.65 105.41)
+		)
+		(stroke
+			(width 0)
+			(type default)
+		)
+	)
+	(wire
+		(pts
 			(xy 217.17 93.98) (xy 237.49 93.98)
 		)
@@
 	(wire
 		(pts
-			(xy 118.11 86.36) (xy 148.59 86.36)
-		)
-		(stroke
-			(width 0)
-			(type default)
-		)
-	)
-	(wire
-		(pts
 			(xy 196.85 116.84) (xy 214.63 116.84)
 		)
@@
 	(wire
 		(pts
+			(xy 252.73 86.36) (xy 245.11 86.36)
+		)
+		(stroke
+			(width 0)
+			(type default)
+		)
+	)
+	(wire
+		(pts
 			(xy 224.79 86.36) (xy 229.87 86.36)
 		)
@@
 	(wire
 		(pts
-			(xy 118.11 124.46) (xy 148.59 124.46)
+			(xy 146.05 86.36) (xy 146.05 105.41)
 		)
 		(stroke
@@
 	(wire
 		(pts
+			(xy 245.11 67.31) (xy 252.73 67.31)
+		)
+		(stroke
+			(width 0)
+			(type default)
+		)
+	)
+	(wire
+		(pts
 			(xy 196.85 93.98) (xy 217.17 93.98)
 		)
@@
 	(wire
 		(pts
-			(xy 118.11 86.36) (xy 118.11 105.41)
-		)
-		(stroke
-			(width 0)
-			(type default)
-		)
-	)
-	(wire
-		(pts
 			(xy 204.47 67.31) (xy 209.55 67.31)
 		)
@@
 	(wire
 		(pts
+			(xy 247.65 124.46) (xy 245.11 124.46)
+		)
+		(stroke
+			(width 0)
+			(type default)
+		)
+	)
+	(wire
+		(pts
 			(xy 224.79 67.31) (xy 229.87 67.31)
 		)
@@
 	(wire
 		(pts
+			(xy 247.65 105.41) (xy 247.65 124.46)
+		)
+		(stroke
+			(width 0)
+			(type default)
+		)
+	)
+	(wire
+		(pts
 			(xy 163.83 124.46) (xy 168.91 124.46)
 		)
@@
 	(wire
 		(pts
+			(xy 252.73 67.31) (xy 252.73 86.36)
+		)
+		(stroke
+			(width 0)
+			(type default)
+		)
+	)
+	(wire
+		(pts
 			(xy 156.21 93.98) (xy 176.53 93.98)
 		)
@@
 	(wire
 		(pts
+			(xy 146.05 105.41) (xy 148.59 105.41)
+		)
+		(stroke
+			(width 0)
+			(type default)
+		)
+	)
+	(wire
+		(pts
 			(xy 194.31 97.79) (xy 196.85 97.79)
 		)
@@
 	(wire
 		(pts
-			(xy 118.11 105.41) (xy 118.11 124.46)
-		)
-		(stroke
-			(width 0)
-			(type default)
-		)
-	)
-	(wire
-		(pts
 			(xy 217.17 59.69) (xy 234.95 59.69)
 		)
@@
 		)
 		(stroke
-			(width 0)
-			(type default)
-		)
-	)
-	(wire
-		(pts
-			(xy 118.11 67.31) (xy 118.11 86.36)
-		)
-		(stroke
